File: hardware/spoke/spoke.sch (EAGLE design)
At the start: 0 parts

Commit message: Put some bits on a schematic
Parts:
- added J1: ICSP, avr-isp:AVR-ISP-6PINAVR-ISP-6PIN-SMALL-SILK
- added U$1: AT25M01DIP'D, aurai:AT25M01DIP'D
- added U1: ATMEGA328P_PDIP, SparkFun-DigitalIC:ATMEGA328P_PDIP
