File: hardware/spoke/spoke.sch (EAGLE design)
At the start: 25 parts, among them IC1 7805TV, J1 AVR_SPI_PRG_6PTH, J2 POWER_JACKPTH, U1 ATMEGA328P_PDIP, U3 NRF24L01+

Commit message: Add real 3.3v LDO regulator
Parts:
- removed 1000: 100, SparkFun-Resistors:RESISTOR0805-RES
- removed 500: 50, SparkFun-Resistors:RESISTOR0805-RES
- added C4: 0.47uF, SparkFun-Capacitors:CAPPTH
- added C5: 33uF, SparkFun-Capacitors:CAPPTH
- added IC3: LM3940, aurai:LM3940
Connections:
- net 3.3V: now also C5.1, IC3.VO; no longer 1000.1, 500.2
- net 5V: now also C4.1, IC3.VI; no longer 500.1
- net GND: now also C4.2, C5.2, IC3.GND; no longer 1000.2
Other:
- note added: "3.3v power supply"
- note removed: "3.3v voltage divider"
Changed lines of the file:
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@@
 <part name="SUPPLY2" library="SparkFun-Aesthetics" deviceset="5V" device=""/>
 <part name="IC1" library="linear" deviceset="78*" device="TV" technology="05"/>
-<part name="500" library="SparkFun-Resistors" deviceset="RESISTOR" device="0805-RES" value="50"/>
-<part name="1000" library="SparkFun-Resistors" deviceset="RESISTOR" device="0805-RES" value="100"/>
-<part name="GND12" library="SparkFun-Aesthetics" deviceset="GND" device=""/>
 <part name="SUPPLY7" library="SparkFun-Aesthetics" deviceset="5V" device=""/>
 <part name="SUPPLY8" library="SparkFun-Aesthetics" deviceset="3.3V" device=""/>
@@
 <part name="R7" library="SparkFun-Resistors" deviceset="RESISTOR" device="0805-RES" value="5k"/>
 <part name="SUPPLY9" library="SparkFun-Aesthetics" deviceset="5V" device=""/>
+<part name="GND6" library="SparkFun-Aesthetics" deviceset="GND" device=""/>
+<part name="C4" library="SparkFun-Capacitors" deviceset="CAP" device="PTH" value="0.47uF"/>
+<part name="C5" library="SparkFun-Capacitors" deviceset="CAP" device="PTH" value="33uF"/>
+<part name="IC3" library="aurai" deviceset="LM3940" device=""/>
 </parts>
 <sheets>
@@
 <wire x1="68.58" y1="132.08" x2="68.58" y2="99.06" width="0.2032" layer="97"/>
 <text x="2.794" y="127.254" size="2.54" layer="97">Programming connection</text>
-<wire x1="68.58" y1="99.06" x2="68.58" y2="63.5" width="0.2032" layer="97"/>
-<wire x1="68.58" y1="63.5" x2="68.58" y2="0" width="0.2032" layer="97"/>
+<wire x1="68.58" y1="99.06" x2="68.58" y2="45.72" width="0.2032" layer="97"/>
+<wire x1="68.58" y1="45.72" x2="68.58" y2="0" width="0.2032" layer="97"/>
 <wire x1="68.58" y1="99.06" x2="0" y2="99.06" width="0.2032" layer="97"/>
-<wire x1="68.58" y1="63.5" x2="0" y2="63.5" width="0.2032" layer="97"/>
-<text x="2.794" y="94.234" size="2.54" layer="97">3.3v voltage divider</text>
+<wire x1="68.58" y1="45.72" x2="0" y2="45.72" width="0.2032" layer="97"/>
+<text x="2.794" y="94.234" size="2.54" layer="97">3.3v power supply</text>
 </plain>
 <instances>
@@
 <instance part="SUPPLY2" gate="G$1" x="60.96" y="165.1" rot="R270"/>
 <instance part="IC1" gate="A1" x="45.72" y="165.1"/>
-<instance part="500" gate="G$1" x="20.32" y="78.74"/>
-<instance part="1000" gate="G$1" x="45.72" y="78.74"/>
-<instance part="GND12" gate="1" x="55.88" y="71.12"/>
-<instance part="SUPPLY7" gate="G$1" x="10.16" y="83.82"/>
-<instance part="SUPPLY8" gate="G$1" x="33.02" y="83.82"/>
+<instance part="SUPPLY7" gate="G$1" x="20.32" y="81.28" rot="R90"/>
+<instance part="SUPPLY8" gate="G$1" x="50.8" y="81.28" rot="R270"/>
 <instance part="R6" gate="G$1" x="195.58" y="83.82" rot="R180"/>
 <instance part="R7" gate="G$1" x="114.3" y="160.02" rot="R90"/>
 <instance part="SUPPLY9" gate="G$1" x="114.3" y="167.64"/>
+<instance part="GND6" gate="1" x="35.56" y="53.34"/>
+<instance part="C4" gate="G$1" x="27.94" y="60.96"/>
+<instance part="C5" gate="G$1" x="43.18" y="60.96"/>
+<instance part="IC3" gate="IC" x="35.56" y="81.28"/>
 </instances>
 <busses>
@@
 </segment>
 <segment>
-<pinref part="1000" gate="G$1" pin="2"/>
-<wire x1="50.8" y1="78.74" x2="55.88" y2="78.74" width="0.1524" layer="91"/>
-<wire x1="55.88" y1="78.74" x2="55.88" y2="73.66" width="0.1524" layer="91"/>
-<pinref part="GND12" gate="1" pin="GND"/>
+<pinref part="GND6" gate="1" pin="GND"/>
+<wire x1="35.56" y1="73.66" x2="35.56" y2="55.88" width="0.1524" layer="91"/>
+<wire x1="43.18" y1="55.88" x2="35.56" y2="55.88" width="0.1524" layer="91"/>
+<junction x="35.56" y="55.88"/>
+<wire x1="35.56" y1="55.88" x2="27.94" y2="55.88" width="0.1524" layer="91"/>
+<wire x1="27.94" y1="55.88" x2="27.94" y2="58.42" width="0.1524" layer="91"/>
+<wire x1="43.18" y1="58.42" x2="43.18" y2="55.88" width="0.1524" layer="91"/>
+<pinref part="C4" gate="G$1" pin="2"/>
+<pinref part="C5" gate="G$1" pin="2"/>
+<pinref part="IC3" gate="IC" pin="GND"/>
+<junction x="35.56" y="73.66"/>
 </segment>
 </net>
@@
 </segment>
 <segment>
-<pinref part="500" gate="G$1" pin="1"/>
-<wire x1="15.24" y1="78.74" x2="10.16" y2="78.74" width="0.1524" layer="91"/>
-<wire x1="10.16" y1="78.74" x2="10.16" y2="83.82" width="0.1524" layer="91"/>
-<pinref part="SUPPLY7" gate="G$1" pin="5V"/>
-</segment>
-<segment>
 <pinref part="SUPPLY9" gate="G$1" pin="5V"/>
 <pinref part="R7" gate="G$1" pin="2"/>
 <wire x1="114.3" y1="167.64" x2="114.3" y2="165.1" width="0.1524" layer="91"/>
 </segment>
+<segment>
+<wire x1="27.94" y1="81.28" x2="25.4" y2="81.28" width="0.1524" layer="91"/>
+<pinref part="C4" gate="G$1" pin="1"/>
+<wire x1="27.94" y1="66.04" x2="27.94" y2="68.58" width="0.1524" layer="91"/>
+<wire x1="27.94" y1="68.58" x2="25.4" y2="68.58" width="0.1524" layer="91"/>
+<wire x1="25.4" y1="68.58" x2="25.4" y2="81.28" width="0.1524" layer="91"/>
+<junction x="25.4" y="81.28"/>
+<pinref part="IC3" gate="IC" pin="VI"/>
+<junction x="25.4" y="81.28"/>
+<wire x1="20.32" y1="81.28" x2="25.4" y2="81.28" width="0.1524" layer="91"/>
+<pinref part="SUPPLY7" gate="G$1" pin="5V"/>
+</segment>
 </net>
 <net name="3.3V" class="0">
-<segment>
-<pinref part="500" gate="G$1" pin="2"/>
-<pinref part="1000" gate="G$1" pin="1"/>
-<wire x1="25.4" y1="78.74" x2="33.02" y2="78.74" width="0.1524" layer="91"/>
-<wire x1="33.02" y1="78.74" x2="40.64" y2="78.74" width="0.1524" layer="91"/>
-<wire x1="33.02" y1="78.74" x2="33.02" y2="83.82" width="0.1524" layer="91"/>
-<junction x="33.02" y="78.74"/>
-<pinref part="SUPPLY8" gate="G$1" pin="3.3V"/>
-</segment>
 <segment>
 <pinref part="U3" gate="U1" pin="VCC"/>
@@
 <wire x1="238.76" y1="60.96" x2="238.76" y2="63.5" width="0.1524" layer="91"/>
 </segment>
-</net>
+<segment>
+<wire x1="43.18" y1="81.28" x2="45.72" y2="81.28" width="0.1524" layer="91"/>
+<wire x1="45.72" y1="81.28" x2="45.72" y2="68.58" width="0.1524" layer="91"/>
+<wire x1="45.72" y1="68.58" x2="43.18" y2="68.58" width="0.1524" layer="91"/>
+<pinref part="C5" gate="G$1" pin="1"/>
+<wire x1="43.18" y1="68.58" x2="43.18" y2="66.04" width="0.1524" layer="91"/>
+<wire x1="45.72" y1="81.28" x2="50.8" y2="81.28" width="0.1524" layer="91"/>
+<junction x="45.72" y="81.28"/>
+<pinref part="IC3" gate="IC" pin="VO"/>
+<junction x="45.72" y="81.28"/>
+<pinref part="SUPPLY8" gate="G$1" pin="3.3V"/>
+</segment>
+</net>

Commit message: Update spoke board
Parts:
- removed IC3: LM3940, aurai:LM3940
- removed R2, R3, R6: 330, SparkFun-Resistors:RESISTOR0805-RES
- added IC2: LM3490, aurai:LM3490
- C1, C2: device SparkFun-Capacitors:CAPPTH -> SparkFun-Capacitors:CAP0805
- C4: value 0.47uF -> 0.1uF; device SparkFun-Capacitors:CAPPTH -> SparkFun-Capacitors:CAP0805
- C5: value 33uF -> 0.1uF; device SparkFun-Capacitors:CAPPTH -> SparkFun-Capacitors:CAP0805
- R1: device SparkFun-Resistors:RESISTOR0805-RES -> aurai:CRA06ES08
Connections:
- removed net N$10: LED1.A, R1.2
- removed net N$11: LED3.A, R3.2
- new net N$1: LED1.A, R1.R3A
- new net N$6: LED3.A, R1.R1A
- net 3.3V: now also IC2.VO; no longer IC3.VO
- net 5V: now also IC2.ENABLE, IC2.VI; no longer IC3.VI
- net GND: now also IC2.GND1; no longer IC3.GND
- net N$12: now also R1.R3B; no longer R1.1
- net N$15: now also R1.R4A; no longer R6.1
- net N$16: now also R1.R4B; no longer R6.2
- net N$3: now also R1.R2B; no longer R2.1
- net N$5: now also R1.R1B; no longer R3.1
- net N$8: now also R1.R2A; no longer R2.2
Other:
- moved on the sheet: C4, C5, JP2, LED1, LED2, LED3
