File: hardware/hub/hub.sch (EAGLE design)
At the start: 0 parts

Commit message: User interface mock
Parts:
- added C1: 0.33uF, SparkFun-Capacitors:CAP0805
- added C2: 0.1uF, SparkFun-Capacitors:CAP0805
- added C3: 22pF, SparkFun-Passives:CAP0805
- added C4: 0.47uF, SparkFun-Capacitors:CAP0805
- added C5: 33uF, SparkFun-Capacitors:CAP0805
- added IC1: 7805TV, linear:7805TV
- added IC2: LM3940, aurai:LM3940
- added J1: AVR_SPI_PRG_6PTH, SparkFun-Connectors:AVR_SPI_PRG_6PTH
- added J2: POWER_JACKPTH, SparkFun-Connectors:POWER_JACKPTH
- added JP1: SERIAL, SparkFun-Connectors:M02PTH
- added LED1: GRN, SparkFun-LED:LED1206
- added LED2: YLW, SparkFun-LED:LED1206
- added LED3: RED, SparkFun-LED:LED1206
- added R1: 330, aurai:CRA06ES08
- added STANDOFF1, STANDOFF2, STANDOFF3, STANDOFF4: STAND-OFF, SparkFun-Electromechanical:STAND-OFF
- added U$1: AT45DB161E-SHD2B-T, aurai:AT45DB161E-SHD2B-T
- added U1: ATMEGA328P_PDIP, SparkFun-DigitalIC:ATMEGA328P_PDIP
- added U2: ENC28J60, aurai:ENC28J60
- added U3: NRF24L01+, aurai:NRF24L01+
Connections:
- new net 3.3V: C5.1, IC2.VO, U$1.!RESET, U$1.!WP, U$1.VCC, U2.VCC, U3.VCC
- new net 5V: C2.1, C3.1, C4.1, IC1.VO, IC2.VI, J1.2, U1.AVCC, U1.VCC
- new net GND: C1.2, C2.2, C3.2, C4.2, C5.2, IC1.GND, IC2.GND, J1.6, J2.GND, J2.GNDBREAK, LED1.C, LED2.C, LED3.C, U$1.GND, U1.GND@1, U2.GND, U3.GND
- new net MISO: J1.1, U$1.MISO, U1.PB4(MISO), U2.MISO, U3.MISO
- new net MOSI: J1.4, U$1.MOSI, U1.PB3(MOSI/OC2), U2.MOSI, U3.MOSI
- new net N$1: LED1.A, R1.R3A
- new net N$10: U1.PD3(INT1), U3.IRQ
- new net N$11: U$1.!CS, U1.PC2(ADC2)
- new net N$12: R1.R3B, U1.PC5(ADC5/SCL)
- new net N$13: U1.PC0(ADC0), U2.!CS
- new net N$14: C1.1, IC1.VI, J2.PWR
- new net N$15: U1.PD2(INT0), U2.INT
- new net N$2: JP1.1, U1.PD0(RXD)
- new net N$3: R1.R2B, U1.PC4(ADC4/SDA)
- new net N$4: JP1.2, U1.PD1(TXD)
- new net N$5: R1.R1B, U1.PC3(ADC3)
- new net N$6: LED3.A, R1.R1A
- new net N$7: U1.PB1(OC1A), U3.!CSN
- new net N$8: LED2.A, R1.R2A
- new net N$9: U1.PB2(SS/OC1B), U3.CE
- new net RESET: J1.5, U1.PC6(/RESET)
- new net SCK: J1.3, U$1.SCK, U1.PB5(SCK), U2.SCK, U3.SCK
Other:
- note added: "3.3v power supply"
- note added: "External Power Supply"
- note added: "Programming connection"
